File: hw/sch_pcb/UST2BATTD01A.kicad_pcb (KiCad board)
At the start: 2 copper layers, 8 parts, among them J1 SM03B-GHS-TB, J2 SM03B-GHS-TB

Commit message: Edit PCB
Parts:
- moved D2 285.7 mm to (160.9, 127.8), turned to 90 degrees
- moved F2 272.9 mm to (161.3, 119.8)
- moved J1 227.7 mm to (161.5, 137.8), turned to 90 degrees
- moved BT2 216.9 mm to (138.4, 106.2), turned to -90 degrees
- moved J2 195.3 mm to (77.2, 137.9), turned to -90 degrees
- moved D1 157.7 mm to (77.3, 127.9), turned to 90 degrees
- moved F1 147.3 mm to (77.1, 121.3)
- moved BT1 57.2 mm to (100.3, 106.2), turned to 90 degrees
Other:
- board outline added: 90.9 x 72 mm

Commit message: Edit PCB
Parts:
- added D3: LSM115JE3/TR13, Diode_SMD:D_SMA_Handsoldering, B.Cu at (160.9, 127.8)
- added D4: LSM115JE3/TR13, Diode_SMD:D_SMA_Handsoldering, B.Cu at (77.3, 127.9)
- added F3: SR010-15, Fuse:Fuse_0805_2012Metric_Pad1.15x1.40mm_HandSolder, B.Cu at (77.1, 121.3)
- added F4: SR010-15, Fuse:Fuse_0805_2012Metric_Pad1.15x1.40mm_HandSolder, B.Cu at (161.3, 119.8)
- added J3: SM03B-GHS-TB, Connector_JST:JST_GH_SM03B-GHS-TB_1x03-1MP_P1.25mm_Horizontal, B.Cu at (161.5, 137.2)
- added J4: SM03B-GHS-TB, Connector_JST:JST_GH_SM03B-GHS-TB_1x03-1MP_P1.25mm_Horizontal, B.Cu at (77.2, 137.2)
- moved J2 0.68 mm to (77.2, 137.2)
- moved J1 0.56 mm to (161.5, 137.2)
- turned BT2 to 90 degrees

Commit message: Edit PCB
Parts:
- moved D4 83.6 mm to (160.9, 127.8)
- moved D3 83.6 mm to (77.3, 127.9)
- turned F2 to 180 degrees
- turned F4 to 180 degrees
Routing:
- net Net-(D1-Pad1): track 0.00 -> 127.5 mm, vias 0 -> 4
- net Net-(F1-Pad2): track 0.00 -> 37.6 mm, vias 0 -> 2
- net Net-(F2-Pad2): track 0.00 -> 37.1 mm, vias 0 -> 2
- net Net-(D4-Pad2): track 0.00 -> 6.08 mm
- net Net-(D2-Pad2): track 0.00 -> 6.08 mm
- net Net-(D3-Pad2): track 0.00 -> 4.63 mm
- net Net-(D1-Pad2): track 0.00 -> 4.63 mm
- added copper zone on B.Cu, net GND
- added copper zone on F.Cu, net GND
Other:
- board text added: "JACHO 2022"
- board text added: "UST.CZ UST2BATTD01A"
- board text removed: "3V6"
- board text removed: "GND"
- board text removed: "OUT"
- board text removed: "UST.CZ USTSIPM01A"
